File: Electronics/lights.kicad_sch (KiCad schematic)
At the start: 42 parts

Commit message: Schematic update
Added correct values for crystal capacitors, added net labels and minor cleanup
Other:
- note added: "12V MAX 2A"
- note removed: "12V @ 2A"
Changed lines of the file:
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@@
     (stroke (width 0) (type default))
   )
-  (text "12V @ 2A" (at 107.95 49.53 0)
+  (text "12V MAX 2A" (at 107.95 49.53 0)
     (effects (font (size 1.27 1.27)) (justify left bottom))
   )

Commit message: Power and lights update
Changed STUSB4500 + BQ25895 to MP2722. Changed Lights power supply, now it's split up to 3 LED drivers - KTD2801 as 10s1p. Added fuses to each battery. Added ESD protection. Fixed CHIP_EN pin name on ESP32-C3 and pull-up resistor on I2C lines.
Parts:
- removed D10, D11, D12, D13, D14, D15, D16, D17, D18, D19, D2, D20, D21, D22, D23, D24, D25, D26, D27, D28, D29, D3, D30, D31, D32, D33, D34, D35, D36, D4, D5, D6, D7, D8, D9: LED, symbol Device:LED
- removed R21, R22, R23, R24, R25, R26, R27: 10R, symbol Device:R
- added C19, C21, C31: 10u, symbol Device:C_Small
- added C20, C22, C32: 470n, symbol Device:C_Small
- added D1, D10, D11, D12, D13, D14, D15, D16, D17, D18, D19, D2, D20, D21, D22, D23, D24, D25, D26, D27, D28, D29, D3, D30, D4, D5, D6, D7, D8, D9: LED, symbol Device:LED_Small
- added L4, L5, L6: 22u, symbol Device:L_Small
- added R7, R8, R9: 1R3, symbol Device:R_Small
- added U7 (x3): KTD2801, Package_DFN_QFN:DFN-6-1EP_2x2mm_P0.65mm_EP1x1.6mm, symbol Drivers_LED:KTD2801
Connections:
- net Earth: now also C19.2, C20.1, C21.2, C22.1, C31.2, C32.1, R7.2, R8.2, R9.2, U7.5 (GND), U7.5 (GND), U7.5 (GND)
- new net: C20.2, D1.2 (A), U7.3 (VOUT)
- new net: D10.1 (K), R7.1, U7.4 (FB)
- new net: L4.2, U7.6 (LX)
- new net: C22.2, D11.2 (A), U7.3 (VOUT)
- new net: D2.1 (K), D3.2 (A)
- new net: D1.1 (K), D2.2 (A)
- new net: D27.1 (K), D28.2 (A)
- new net: D26.1 (K), D27.2 (A)
- new net: D20.1 (K), R8.1, U7.4 (FB)
- new net: L5.2, U7.6 (LX)
- new net: D8.1 (K), D9.2 (A)
- new net: D7.1 (K), D8.2 (A)
- new net: D6.1 (K), D7.2 (A)
- new net: D29.1 (K), D30.2 (A)
- new net: D28.1 (K), D29.2 (A)
- new net: D4.1 (K), D5.2 (A)
- new net: D3.1 (K), D4.2 (A)
- new net: D11.1 (K), D12.2 (A)
- new net: D13.1 (K), D14.2 (A)
- new net: D12.1 (K), D13.2 (A)
- new net: D21.1 (K), D22.2 (A)
- new net: C32.2, D21.2 (A), U7.3 (VOUT)
- new net: L6.2, U7.6 (LX)
- new net: D18.1 (K), D19.2 (A)
- new net: D17.1 (K), D18.2 (A)
- new net: D10.2 (A), D9.1 (K)
- new net: D22.1 (K), D23.2 (A)
- new net: D19.1 (K), D20.2 (A)
- new net: D30.1 (K), R9.1, U7.4 (FB)
- new net: D16.1 (K), D17.2 (A)
- new net: D24.1 (K), D25.2 (A)
- new net: D23.1 (K), D24.2 (A)
- new net: D5.1 (K), D6.2 (A)
- new net: D25.1 (K), D26.2 (A)
- new net: D14.1 (K), D15.2 (A)
- new net: D15.1 (K), D16.2 (A)
- new net L_CONT: U7.1 (CTRL), U7.1 (CTRL), U7.1 (CTRL)
- new net VSYS: C19.1, C21.1, C31.1, L4.1, L5.1, L6.1, U7.2 (VIN), U7.2 (VIN), U7.2 (VIN)
Other:
- note added: "LEDs used: Red JE2835 Max current: 250mA Target current: 140-200mA Forward voltage: 2.2V"
- note added: "R = 200mV / I_{MAX}"
- note removed: "12V MAX 2A"
- note removed: "LEDs used: Red JE2835 Max current: 250mA Target current: 160-200mA Forward voltage: 2.2V"

Commit message: PCB Layout mostly completed
Still have to finish LEDs layout on back side
Parts:
- C19, C21, C31: footprint (none) -> Capacitor_SMD:C_0603_1608Metric
- C20, C22, C32: footprint (none) -> Capacitor_SMD:C_0805_2012Metric
- D1, D10, D11, D12, D13, D14, D15, D16, D17, D18, D19, D2, D20, D21, D22, D23, D24, D25, D26, D27, D28, D29, D3, D30, D4, D5, D6, D7, D8, D9: footprint (none) -> SMD-1411:LED_EAHC2835WD6
- L4, L5, L6: value 22u -> 10u; footprint (none) -> SMD 1616:IND_XFL4020-102MEC
- R7, R8, R9: footprint (none) -> Resistor_SMD:R_0805_2012Metric
