File: Electronics/sensors.kicad_sch (KiCad schematic)
At the start: 14 parts, among them U4 LIS3MDL, U5 LSM6DS3

Commit message: Schematic update
Added correct values for crystal capacitors, added net labels and minor cleanup
Connections:
- net Earth: now also U4.12 (GND), U4.2 (GND), U4.3 (GND)
- net ACC_ADD: now reaches JP1.2 (B), R16.2, U5.1 (SDO/SA0)
- net MAG_ADD: now reaches JP2.2 (B), R18.2, U4.9 (SDO/SA1)
Changed lines of the file:
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@@
   (no_connect (at 129.54 48.26))
   (no_connect (at 69.85 49.53))
+  (wire (pts (xy 21.59 60.96) (xy 21.59 59.69))
+    (stroke (width 0) (type default))
+  )
+  (wire (pts (xy 121.92 67.31) (xy 124.46 67.31))
+    (stroke (width 0) (type default))
+  )
+  (wire (pts (xy 72.39 62.23) (xy 72.39 64.77))
+    (stroke (width 0) (type default))
+  )
+  (wire (pts (xy 31.75 29.21) (xy 31.75 30.48))
+    (stroke (width 0) (type default))
+  )
+  (wire (pts (xy 114.3 67.31) (xy 114.3 66.04))
+    (stroke (width 0) (type default))
+  )
+  (wire (pts (xy 31.75 30.48) (xy 43.18 30.48))
+    (stroke (width 0) (type default))
+  )
+  (wire (pts (xy 105.41 38.1) (xy 116.84 38.1))
+    (stroke (width 0) (type default))
+  )
+  (wire (pts (xy 105.41 36.83) (xy 105.41 38.1))
+    (stroke (width 0) (type default))
+  )
+  (wire (pts (xy 124.46 60.96) (xy 129.54 60.96))
+    (stroke (width 0) (type default))
+  )
+  (wire (pts (xy 105.41 45.72) (xy 129.54 45.72))
+    (stroke (width 0) (type default))
+  )
+  (wire (pts (xy 100.33 45.72) (xy 105.41 45.72))
+    (stroke (width 0) (type default))
+  )
+  (wire (pts (xy 144.78 35.56) (xy 147.32 35.56))
+    (stroke (width 0) (type default))
+  )
+  (wire (pts (xy 57.15 36.83) (xy 59.69 36.83))
+    (stroke (width 0) (type default))
+  )
+  (wire (pts (xy 43.18 38.1) (xy 31.75 38.1))
+    (stroke (width 0) (type default))
+  )
+  (wire (pts (xy 31.75 71.12) (xy 31.75 73.66))
+    (stroke (width 0) (type default))
+  )
+  (wire (pts (xy 35.56 60.96) (xy 35.56 54.61))
+    (stroke (width 0) (type default))
+  )
+  (wire (pts (xy 144.78 69.85) (xy 144.78 68.58))
+    (stroke (width 0) (type default))
+  )
+  (wire (pts (xy 22.86 46.99) (xy 21.59 46.99))
+    (stroke (width 0) (type default))
+  )
+  (wire (pts (xy 105.41 30.48) (xy 105.41 31.75))
+    (stroke (width 0) (type default))
+  )
+  (wire (pts (xy 22.86 60.96) (xy 21.59 60.96))
+    (stroke (width 0) (type default))
+  )
+  (wire (pts (xy 105.41 55.88) (xy 105.41 58.42))
+    (stroke (width 0) (type default))
+  )
+  (wire (pts (xy 105.41 30.48) (xy 116.84 30.48))
+    (stroke (width 0) (type default))
+  )
+  (wire (pts (xy 116.84 30.48) (xy 128.27 30.48))
+    (stroke (width 0) (type default))
+  )
   (wire (pts (xy 35.56 54.61) (xy 44.45 54.61))
     (stroke (width 0) (type default))
   )
-  (wire (pts (xy 21.59 60.96) (xy 21.59 59.69))
-    (stroke (width 0) (type default))
-  )
-  (wire (pts (xy 121.92 67.31) (xy 124.46 67.31))
-    (stroke (width 0) (type default))
-  )
-  (wire (pts (xy 72.39 62.23) (xy 72.39 64.77))
-    (stroke (width 0) (type default))
-  )
-  (wire (pts (xy 31.75 29.21) (xy 31.75 30.48))
-    (stroke (width 0) (type default))
-  )
-  (wire (pts (xy 114.3 67.31) (xy 114.3 66.04))
-    (stroke (width 0) (type default))
-  )
-  (wire (pts (xy 31.75 30.48) (xy 43.18 30.48))
-    (stroke (width 0) (type default))
-  )
-  (wire (pts (xy 105.41 38.1) (xy 116.84 38.1))
-    (stroke (width 0) (type default))
-  )
-  (wire (pts (xy 105.41 36.83) (xy 105.41 38.1))
-    (stroke (width 0) (type default))
-  )
-  (wire (pts (xy 124.46 60.96) (xy 129.54 60.96))
-    (stroke (width 0) (type default))
-  )
-  (wire (pts (xy 105.41 45.72) (xy 129.54 45.72))
-    (stroke (width 0) (type default))
-  )
-  (wire (pts (xy 100.33 45.72) (xy 105.41 45.72))
-    (stroke (width 0) (type default))
-  )
-  (wire (pts (xy 144.78 35.56) (xy 147.32 35.56))
-    (stroke (width 0) (type default))
-  )
-  (wire (pts (xy 57.15 36.83) (xy 59.69 36.83))
-    (stroke (width 0) (type default))
-  )
-  (wire (pts (xy 43.18 38.1) (xy 31.75 38.1))
-    (stroke (width 0) (type default))
-  )
-  (wire (pts (xy 31.75 71.12) (xy 31.75 73.66))
-    (stroke (width 0) (type default))
-  )
-  (wire (pts (xy 35.56 60.96) (xy 35.56 54.61))
-    (stroke (width 0) (type default))
-  )
-  (wire (pts (xy 144.78 69.85) (xy 144.78 68.58))
-    (stroke (width 0) (type default))
-  )
-  (wire (pts (xy 22.86 46.99) (xy 21.59 46.99))
-    (stroke (width 0) (type default))
-  )
-  (wire (pts (xy 105.41 30.48) (xy 105.41 31.75))
-    (stroke (width 0) (type default))
-  )
-  (wire (pts (xy 22.86 60.96) (xy 21.59 60.96))
-    (stroke (width 0) (type default))
-  )
-  (wire (pts (xy 105.41 55.88) (xy 105.41 58.42))
-    (stroke (width 0) (type default))
-  )
-  (wire (pts (xy 105.41 30.48) (xy 116.84 30.48))
-    (stroke (width 0) (type default))
-  )
-  (wire (pts (xy 116.84 30.48) (xy 128.27 30.48))
-    (stroke (width 0) (type default))
-  )
   (wire (pts (xy 31.75 38.1) (xy 31.75 36.83))
     (stroke (width 0) (type default))
@@
     (stroke (width 0) (type default))
   )
+  (wire (pts (xy 57.15 67.31) (xy 57.15 64.77))
+    (stroke (width 0) (type default))
+  )
   (wire (pts (xy 72.39 54.61) (xy 72.39 57.15))
     (stroke (width 0) (type default))
@@
     (stroke (width 0) (type default))
   )
-  (wire (pts (xy 41.91 52.07) (xy 44.45 52.07))
-    (stroke (width 0) (type default))
-  )
-  (wire (pts (xy 41.91 49.53) (xy 44.45 49.53))
+  (wire (pts (xy 36.83 52.07) (xy 44.45 52.07))
+    (stroke (width 0) (type default))
+  )
+  (wire (pts (xy 36.83 49.53) (xy 44.45 49.53))
     (stroke (width 0) (type default))
   )
@@
     (effects (font (size 2.5 2.5) (thickness 0.5) bold) (justify left top))
   )
+  (label "MAG_ADD" (at 41.91 54.61 180) (fields_autoplaced)
+    (effects (font (size 0.75 0.75)) (justify right bottom))
+  )
+  (label "ACC_ADD" (at 127 45.72 180) (fields_autoplaced)
+    (effects (font (size 0.75 0.75)) (justify right bottom))
+  )
   (global_label "SCL" (shape passive) (at 127 55.88 180) (fields_autoplaced)
     (effects (font (size 1.27 1.27)) (justify right))
@@
     )
   )
-  (global_label "SDA" (shape bidirectional) (at 41.91 52.07 180) (fields_autoplaced)
+  (global_label "SDA" (shape bidirectional) (at 36.83 52.07 180) (fields_autoplaced)
     (effects (font (size 1.27 1.27)) (justify right))
-    (property "Intersheetrefs" "${INTERSHEET_REFS}" (at 34.3248 52.07 0)
+    (property "Intersheetrefs" "${INTERSHEET_REFS}" (at 29.2448 52.07 0)
       (effects (font (size 1.27 1.27)) (justify right) hide)
     )
   )
-  (global_label "SCL" (shape passive) (at 41.91 49.53 180) (fields_autoplaced)
+  (global_label "SCL" (shape passive) (at 36.83 49.53 180) (fields_autoplaced)
     (effects (font (size 1.27 1.27)) (justify right))
-    (property "Intersheetrefs" "${INTERSHEET_REFS}" (at 36.6079 49.53 0)
+    (property "Intersheetrefs" "${INTERSHEET_REFS}" (at 31.5279 49.53 0)
       (effects (font (size 1.27 1.27)) (justify right) hide)
     )
@@
         (path "/b70621e2-23d0-406f-b359-5b7c90496935/c228e0ec-4506-45b3-97db-8d8d26d6b0c7"
           (reference "C27") (unit 1)
+        )
+      )
+    )
+  )
+  (symbol (lib_id "power:Earth") (at 57.15 67.31 0) (unit 1)
+    (in_bom yes) (on_board yes) (dnp no) (fields_autoplaced)
+    (property "Reference" "#PWR071" (at 57.15 73.66 0)
+      (effects (font (size 1.27 1.27)) hide)
+    )
+    (property "Value" "Earth" (at 57.15 71.12 0)
+      (effects (font (size 1.27 1.27)) hide)
+    )
+    (property "Footprint" "" (at 57.15 67.31 0)
+      (effects (font (size 1.27 1.27)) hide)
+    )
+    (property "Datasheet" "~" (at 57.15 67.31 0)
+      (effects (font (size 1.27 1.27)) hide)
+    )
+    (pin "1")
+    (instances
+      (project "Aitken"
+        (path "/b70621e2-23d0-406f-b359-5b7c90496935/c228e0ec-4506-45b3-97db-8d8d26d6b0c7"
+          (reference "#PWR071") (unit 1)
         )
       )
@@
   )
   (symbol (lib_id "Sensor_Magnetic:LIS3MDL") (at 57.15 52.07 0) (unit 1)
-    (in_bom yes) (on_board yes) (dnp no) (fields_autoplaced)
-    (property "Reference" "U4" (at 59.1059 64.77 0)
-      (effects (font (size 1.27 1.27)) (justify left))
-    )
-    (property "Value" "LIS3MDL" (at 59.1059 67.31 0)
-      (effects (font (size 1.27 1.27)) (justify left))
-    )
+    (in_bom yes) (on_board yes) (dnp no)
+    (property "Reference" "U4" (at 64.77 63.5 0)
+      (effects (font (size 1.27 1.27)) (justify left))
+    )
+    (property "Value" "LIS3MDL" (at 46.99 63.5 0)
+      (effects (font (size 1.27 1.27)) (justify left))
+    )

Commit message: PCB Layout mostly completed
Still have to finish LEDs layout on back side
Parts:
- removed C25: 1u, symbol Device:C_Small
- C23, C24, C27, C28: footprint (none) -> Capacitor_SMD:C_0402_1005Metric
- C26: footprint (none) -> Capacitor_SMD:CP_Elec_4x4.5
- JP1, JP2: footprint (none) -> Jumper:SolderJumper-2_P1.3mm_Open_Pad1.0x1.5mm
- R15, R16, R17, R18: footprint (none) -> Resistor_SMD:R_0402_1005Metric
Changed lines of the file:
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@@
     (company "b1u3-22")
   )
-  (junction (at 105.41 38.1) (diameter 0) (color 0 0 0 0)
-  )
   (junction (at 31.75 60.96) (diameter 0) (color 0 0 0 0)
   )
   (junction (at 116.84 38.1) (diameter 0) (color 0 0 0 0)
-  )
-  (junction (at 105.41 30.48) (diameter 0) (color 0 0 0 0)
   )
   (junction (at 144.78 35.56) (diameter 0) (color 0 0 0 0)
@@
     (stroke (width 0) (type default))
   )
-  (wire (pts (xy 105.41 38.1) (xy 116.84 38.1))
-    (stroke (width 0) (type default))
-  )
-  (wire (pts (xy 105.41 36.83) (xy 105.41 38.1))
+  (wire (pts (xy 114.3 38.1) (xy 116.84 38.1))
     (stroke (width 0) (type default))
   )
@@
     (stroke (width 0) (type default))
   )
-  (wire (pts (xy 105.41 30.48) (xy 105.41 31.75))
-    (stroke (width 0) (type default))
-  )
   (wire (pts (xy 22.86 60.96) (xy 21.59 60.96))
     (stroke (width 0) (type default))
@@
     (stroke (width 0) (type default))
   )
-  (wire (pts (xy 105.41 30.48) (xy 116.84 30.48))
+  (wire (pts (xy 114.3 30.48) (xy 116.84 30.48))
     (stroke (width 0) (type default))
   )
@@
     (stroke (width 0) (type default))
   )
-  (wire (pts (xy 105.41 29.21) (xy 105.41 30.48))
+  (wire (pts (xy 114.3 29.21) (xy 114.3 30.48))
     (stroke (width 0) (type default))
   )
@@
     (stroke (width 0) (type default))
   )
-  (wire (pts (xy 105.41 38.1) (xy 105.41 39.37))
+  (wire (pts (xy 114.3 38.1) (xy 114.3 39.37))
     (stroke (width 0) (type default))
   )
@@
       (effects (font (size 1.27 1.27)) (justify left))
     )
-    (property "Footprint" "" (at 72.39 59.69 0)
+    (property "Footprint" "Capacitor_SMD:C_0402_1005Metric" (at 72.39 59.69 0)
       (effects (font (size 1.27 1.27)) hide)
     )
@@
       (effects (font (size 1.27 1.27)) (justify left))
     )
-    (property "Footprint" "" (at 119.38 67.31 0)
+    (property "Footprint" "Resistor_SMD:R_0402_1005Metric" (at 119.38 67.31 0)
       (effects (font (size 1.27 1.27)) hide)
     )
@@
       (effects (font (size 1.27 1.27)) (justify left))
     )
-    (property "Footprint" "" (at 25.4 46.99 0)
+    (property "Footprint" "Resistor_SMD:R_0402_1005Metric" (at 25.4 46.99 0)
       (effects (font (size 1.27 1.27)) hide)
     )
@@
       (effects (font (size 1.27 1.27)) (justify right))
     )
-    (property "Footprint" "" (at 105.41 52.07 0)
+    (property "Footprint" "Jumper:SolderJumper-2_P1.3mm_Open_Pad1.0x1.5mm" (at 105.41 52.07 0)
       (effects (font (size 1.27 1.27)) hide)
     )
@@
       (effects (font (size 1.27 1.27)) (justify left))
     )
-    (property "Footprint" "" (at 43.18 34.29 0)
+    (property "Footprint" "Capacitor_SMD:C_0402_1005Metric" (at 43.18 34.29 0)
       (effects (font (size 1.27 1.27)) hide)
     )
@@
     )
   )
-  (symbol (lib_id "power:Earth") (at 105.41 39.37 0) (unit 1)
-    (in_bom yes) (on_board yes) (dnp no) (fields_autoplaced)
-    (property "Reference" "#PWR033" (at 105.41 45.72 0)
-      (effects (font (size 1.27 1.27)) hide)
-    )
-    (property "Value" "Earth" (at 105.41 43.18 0)
-      (effects (font (size 1.27 1.27)) hide)
-    )
-    (property "Footprint" "" (at 105.41 39.37 0)
-      (effects (font (size 1.27 1.27)) hide)
-    )
-    (property "Datasheet" "~" (at 105.41 39.37 0)
+  (symbol (lib_id "power:Earth") (at 114.3 39.37 0) (unit 1)
+    (in_bom yes) (on_board yes) (dnp no) (fields_autoplaced)
+    (property "Reference" "#PWR033" (at 114.3 45.72 0)
+      (effects (font (size 1.27 1.27)) hide)
+    )
+    (property "Value" "Earth" (at 114.3 43.18 0)
+      (effects (font (size 1.27 1.27)) hide)
+    )
+    (property "Footprint" "" (at 114.3 39.37 0)
+      (effects (font (size 1.27 1.27)) hide)
+    )
+    (property "Datasheet" "~" (at 114.3 39.37 0)
       (effects (font (size 1.27 1.27)) hide)
     )
@@
       (effects (font (size 1.27 1.27)) (justify left))
     )
-    (property "Footprint" "" (at 116.84 34.29 0)
+    (property "Footprint" "Capacitor_SMD:C_0402_1005Metric" (at 116.84 34.29 0)
       (effects (font (size 1.27 1.27)) hide)
     )
@@
       (effects (font (size 1.27 1.27)) (justify left))
     )
-    (property "Footprint" "" (at 31.75 34.29 0)
+    (property "Footprint" "Capacitor_SMD:CP_Elec_4x4.5" (at 31.75 34.29 0)
       (effects (font (size 1.27 1.27)) hide)
     )
@@
     )
   )
-  (symbol (lib_id "power:+3V3") (at 105.41 29.21 0) (unit 1)
-    (in_bom yes) (on_board yes) (dnp no) (fields_autoplaced)
-    (property "Reference" "#PWR032" (at 105.41 33.02 0)
-      (effects (font (size 1.27 1.27)) hide)
-    )
-    (property "Value" "+3V3" (at 105.41 25.4 0)
+  (symbol (lib_id "power:+3V3") (at 114.3 29.21 0) (unit 1)
+    (in_bom yes) (on_board yes) (dnp no) (fields_autoplaced)
+    (property "Reference" "#PWR032" (at 114.3 33.02 0)
+      (effects (font (size 1.27 1.27)) hide)
+    )
+    (property "Value" "+3V3" (at 114.3 25.4 0)
       (effects (font (size 1.27 1.27)))
     )
-    (property "Footprint" "" (at 105.41 29.21 0)
-      (effects (font (size 1.27 1.27)) hide)
-    )
-    (property "Datasheet" "" (at 105.41 29.21 0)
+    (property "Footprint" "" (at 114.3 29.21 0)
+      (effects (font (size 1.27 1.27)) hide)
+    )
+    (property "Datasheet" "" (at 114.3 29.21 0)
       (effects (font (size 1.27 1.27)) hide)
     )
@@
       (effects (font (size 1.27 1.27)) (justify left))
     )
-    (property "Footprint" "" (at 97.79 45.72 0)
+    (property "Footprint" "Resistor_SMD:R_0402_1005Metric" (at 97.79 45.72 0)
       (effects (font (size 1.27 1.27)) hide)
     )
@@
       (effects (font (size 1.27 1.27)) (justify left))
     )
-    (property "Footprint" "" (at 128.27 34.29 0)
+    (property "Footprint" "Capacitor_SMD:C_0402_1005Metric" (at 128.27 34.29 0)
       (effects (font (size 1.27 1.27)) hide)
     )
@@
       (effects (font (size 1.27 1.27)) (justify left))
     )
-    (property "Footprint" "" (at 25.4 60.96 0)
+    (property "Footprint" "Resistor_SMD:R_0402_1005Metric" (at 25.4 60.96 0)
       (effects (font (size 1.27 1.27)) hide)
     )
@@
       (effects (font (size 1.27 1.27)) (justify right))
     )
-    (property "Footprint" "" (at 31.75 67.31 0)
+    (property "Footprint" "Jumper:SolderJumper-2_P1.3mm_Open_Pad1.0x1.5mm" (at 31.75 67.31 0)
       (effects (font (size 1.27 1.27)) hide)
     )
@@
         )
       )
-    )
-  )
-  (symbol (lib_id "Device:C_Small") (at 105.41 34.29 0) (unit 1)
-    (in_bom yes) (on_board yes) (dnp no) (fields_autoplaced)
-    (property "Reference" "C25" (at 107.95 33.6613 0)
-      (effects (font (size 1.27 1.27)) (justify left))
-    )
-    (property "Value" "1u" (at 107.95 36.2013 0)
-      (effects (font (size 1.27 1.27)) (justify left))
-    )
-    (property "Footprint" "" (at 105.41 34.29 0)
-      (effects (font (size 1.27 1.27)) hide)
-    )
-    (property "Datasheet" "~" (at 105.41 34.29 0)
-      (effects (font (size 1.27 1.27)) hide)
-    )
-    (pin "1")
-    (pin "2")
-    (instances
-      (project "Aitken"
-        (path "/b70621e2-23d0-406f-b359-5b7c90496935/c228e0ec-4506-45b3-97db-8d8d26d6b0c7"
-          (reference "C25") (unit 1)
-        )
-      )
