File: Electronics/power.kicad_sch (KiCad schematic)
At the start: 44 parts, among them J1 USB_C_Receptacle_USB2.0, Q1 AON3419, Q2 AON3419, SW1 ON_OFF_SWITCH, U2 STUSB4500QTR, U3 BQ25895RTW, U6 NCP186AMX330TAG, U7 MIC2250

Commit message: All schematics complete
Completed battery, power-path and USB-PD management. 3V3 and V_LIGHTS rail. ESP32-C3 together with Magnetometer, Accelerometer and Gyroscope. And the LED lights
Parts:
- removed SW1: ON_OFF_SWITCH, symbol Switch:SW_Push_SPDT
Connections:
- net VSYS: now also C19.1, C20.1, L3.2, U3.15 (SYS), U3.16 (SYS)
- no-connect marks 18 -> 17
Changed lines of the file:
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@@
   (no_connect (at 48.26 152.4))
   (no_connect (at 46.99 88.9))
-  (no_connect (at 124.46 142.24))
   (no_connect (at 48.26 162.56))
   (wire (pts (xy 201.93 49.53) (xy 201.93 40.64))
@@
     (stroke (width 0) (type default))
   )
-  (wire (pts (xy 124.46 137.16) (xy 143.51 137.16))
-    (stroke (width 0) (type default))
-  )
   (wire (pts (xy 134.62 49.53) (xy 140.97 49.53))
     (stroke (width 0) (type default))
@@
   )
   (wire (pts (xy 80.01 170.18) (xy 80.01 171.45))
+    (stroke (width 0) (type default))
+  )
+  (wire (pts (xy 133.35 139.7) (xy 133.35 138.43))
     (stroke (width 0) (type default))
   )
@@
     (stroke (width 0) (type default))
   )
-  (wire (pts (xy 143.51 137.16) (xy 143.51 135.89))
-    (stroke (width 0) (type default))
-  )
   (wire (pts (xy 201.93 87.63) (xy 204.47 87.63))
     (stroke (width 0) (type default))
@@
     (stroke (width 0) (type default))
   )
-  (wire (pts (xy 101.6 139.7) (xy 114.3 139.7))
+  (wire (pts (xy 101.6 139.7) (xy 133.35 139.7))
     (stroke (width 0) (type default))
   )
@@
   )
   (text_box "Powerpath and battery management"
-    (at 17.78 119.38 0) (size 139.7 68.58)
+    (at 17.78 119.38 0) (size 123.19 68.58)
     (stroke (width 0) (type dash))
     (fill (type none))
@@
     (effects (font (size 0.7 0.7) bold) (justify left bottom))
   )
+  (text "3V5 - 4V5" (at 118.11 142.24 0)
+    (effects (font (size 1.27 1.27) bold) (justify left bottom))
+  )
   (text "Recommended value for R_{1} at 12V output is 240k \nR_{2} value can be calculated as R_{2} = R_{1} / ((V_{OUT} / 1.24) - 1)"
     (at 229.87 30.48 0)
     (effects (font (size 0.75 0.75)) (justify left bottom))
-  )
-  (text "3V5 - 4V5" (at 128.27 139.7 0)
-    (effects (font (size 1.27 1.27) bold) (justify left bottom))
   )
   (text "D+ and D- pins are not used\nAll the settings are handled from MCU through I2C\nIt's recommended to disable D+/D- detection together\nwith Maxcharge and HVDCP in the REG02 register"
@@
         (path "/b70621e2-23d0-406f-b359-5b7c90496935/b637dce6-9faa-48d7-ac20-34c7af1e210c"
           (reference "L4") (unit 1)
-        )
-      )
-    )
-  )
-  (symbol (lib_id "more_power:VSYS") (at 143.51 135.89 0) (unit 1)
-    (in_bom yes) (on_board yes) (dnp no) (fields_autoplaced)
-    (property "Reference" "#PWR043" (at 143.51 139.7 0)
-      (effects (font (size 1.27 1.27)) hide)
-    )
-    (property "Value" "VSYS" (at 143.51 132.08 0)
-      (effects (font (size 1.27 1.27)))
-    )
-    (property "Footprint" "" (at 143.51 135.89 0)
-      (effects (font (size 1.27 1.27)) hide)
-    )
-    (property "Datasheet" "" (at 143.51 135.89 0)
-      (effects (font (size 1.27 1.27)) hide)
-    )
-    (pin "1")
-    (instances
-      (project "Aitken"
-        (path "/b70621e2-23d0-406f-b359-5b7c90496935/b637dce6-9faa-48d7-ac20-34c7af1e210c"
-          (reference "#PWR043") (unit 1)
         )
       )
@@
     )
   )
-  (symbol (lib_id "Switch:SW_Push_SPDT") (at 119.38 139.7 0) (unit 1)
-    (in_bom yes) (on_board yes) (dnp no)
-    (property "Reference" "SW1" (at 119.38 132.08 0)
-      (effects (font (size 1.27 1.27)))
-    )
-    (property "Value" "ON_OFF_SWITCH" (at 119.38 134.62 0)
-      (effects (font (size 1.27 1.27)))
-    )
-    (property "Footprint" "" (at 119.38 139.7 0)
-      (effects (font (size 1.27 1.27)) hide)
-    )
-    (property "Datasheet" "~" (at 119.38 139.7 0)
-      (effects (font (size 1.27 1.27)) hide)
-    )
-    (pin "1")
-    (pin "2")
-    (pin "3")
-    (instances
-      (project "Aitken"
-        (path "/b70621e2-23d0-406f-b359-5b7c90496935/b637dce6-9faa-48d7-ac20-34c7af1e210c"
-          (reference "SW1") (unit 1)
-        )
-      )
-    )
-  )
   (symbol (lib_id "power:Earth") (at 113.03 59.69 0) (unit 1)
     (in_bom yes) (on_board yes) (dnp no) (fields_autoplaced)
@@
         )
       )
+    )
+  )
+  (symbol (lib_id "more_power:VSYS") (at 133.35 138.43 0) (unit 1)
+    (in_bom yes) (on_board yes) (dnp no) (fields_autoplaced)
+    (property "Reference" "#PWR043" (at 133.35 142.24 0)
+      (effects (font (size 1.27 1.27)) hide)
+    )
+    (property "Value" "VSYS" (at 133.35 134.62 0)
+      (effects (font (size 1.27 1.27)))
+    )
+    (property "Footprint" "" (at 133.35 138.43 0)
+      (effects (font (size 1.27 1.27)) hide)
+    )
+    (property "Datasheet" "" (at 133.35 138.43 0)
+      (effects (font (size 1.27 1.27)) hide)
+    )
+    (pin "1")
+    (instances
+      (project "Aitken"
+        (path "/b70621e2-23d0-406f-b359-5b7c90496935/b637dce6-9faa-48d7-ac20-34c7af1e210c"
+          (reference "#PWR043") (unit 1)
+        )
+      )

Commit message: Schematic update
Added correct values for crystal capacitors, added net labels and minor cleanup
Parts:
- added TP1: TP_VBUS_DIR, symbol Connector:TestPoint_Small
- added TP2: TP_VBUS, symbol Connector:TestPoint_Small
- added TP3: TP_VLIGHTS, symbol Connector:TestPoint_Small
- added TP4: TP_L_CONT, symbol Connector:TestPoint_Small
- added TP5: TP_3V3, symbol Connector:TestPoint_Small
- added TP6: TP_VSYS, symbol Connector:TestPoint_Small
- added TP7: TP_BATT, symbol Connector:TestPoint_Small
Connections:
- net +3V3: now also TP5.1
- net L_CONT: now also TP4.1
- net VBUS: now also TP1.1, TP2.1; no longer C14.1, Q1.3 (S), Q2.3 (S), R4.1, U2.24 (VDD)
- net VLIGHTS: now also TP3.1
- net VSYS: now also C18.1, L3.1, U3.19 (SW), U3.20 (SW), TP6.1
- net BATT: now reaches BT1.1 (+), BT2.1 (+), C22.1, U3.13 (BAT), U3.14 (BAT)
- net BATT: now also TP7.1
- net BATT_THERM: now reaches R12.1, R13.1, TH1.1, U3.11 (TS)
- net 3V3_FEEDBACK: now reaches C32.2, R19.2, R20.1, U7.1 (FB)
- net VBUS_EN: now reaches R3.2, U2.16 (VBUS_EN_SNK)
- net VBUS_RES: now reaches R7.2, U2.6 (RESET)
- net VBUS_MON: now reaches R6.2, U2.9 (DISCH)
- net BATT_ILIM: now reaches R14.1, U3.10 (ILIM)
- new net: C14.1, Q1.3 (S), Q2.3 (S), R4.1, U2.24 (VDD)
- no-connect marks 17 -> 18
Other:
- note removed: "Either 120R resistor or directly to ground"
- moved on the sheet: BT1, BT2, R7

Commit message: Power and lights update
Changed STUSB4500 + BQ25895 to MP2722. Changed Lights power supply, now it's split up to 3 LED drivers - KTD2801 as 10s1p. Added fuses to each battery. Added ESD protection. Fixed CHIP_EN pin name on ESP32-C3 and pull-up resistor on I2C lines.
Parts:
- removed C19, C20, C22, C31: 10u, symbol Device:C_Small
- removed C21: 47n, symbol Device:C_Small
- removed C32: 2n2, symbol Device:C_Small
- removed C33: 2u2, symbol Device:C_Small
- removed D1: LS4148, symbol Device:D
- removed L3: 2u2, symbol Device:L_Small
- removed L4: 10u, symbol Device:L
- removed Q1, Q2: AON3419, symbol Simulation_SPICE:PMOS
- removed R10, R11: 100k, symbol Device:R_Small
- removed R12: 30k1, symbol Device:R_Small
- removed R13: 5k23, symbol Device:R_Small
- removed R14: 120, symbol Device:R_Small
- removed R19: 240k, symbol Device:R_Small
- removed R20: 27k7, symbol Device:R_Small
- removed R7: 10k, symbol Device:R_Small
- removed R8: 1k, symbol Device:R_Small
- removed R9: 470, symbol Device:R_Small
- removed TH1: Thermistor, symbol Device:Thermistor
- removed TP2: TP_VBUS, symbol Connector:TestPoint_Small
- removed TP3: TP_VLIGHTS, symbol Connector:TestPoint_Small
- removed TP4: TP_L_CONT, symbol Connector:TestPoint_Small
- removed TP6: TP_VSYS, symbol Connector:TestPoint_Small
- removed TP7: TP_BATT, symbol Connector:TestPoint_Small
- removed U2: STUSB4500QTR, Package_DFN_QFN:QFN-24-1EP_4x4mm_P0.5mm_EP2.7x2.7mm, symbol Interface_USB:STUSB4500QTR
- removed U3: BQ25895RTW, Package_DFN_QFN:Texas_S-PWQFN-N24_EP2.7x2.7mm_ThermalVias, symbol Battery_Management:BQ25895RTW
- removed U7: MIC2250, Package_DFN_QFN:Micrel_MLF-8-1EP_2x2mm_P0.5mm_EP0.6x1.2mm, symbol Regulators_Switching:MIC2250
- added D37: SMF22CA, symbol Device:D_TVS
- added F1: F_BATT_1, symbol Device:Fuse_Small
- added F2: F_BATT_2, symbol Device:Fuse_Small
- added L3: 1u, symbol Device:L
- added TH1: BATT_TEMP, symbol Device:Thermistor_NTC
- added U2: MP2722, QFN-22:MP2722GRH0000Z, symbol Battery_ICs:MP2722
- added U3: TPD4E02B04DQA, Package_SON:USON-10_2.5x1.0mm_P0.5mm, symbol Power_Protection:TPD4E02B04DQA
- C12, C16, C17: value 1u -> 10u
- C14: value 1u -> 4u7
- C15: value 100n -> 22n
- C18: value 47n -> 10u
- R3: value 22k -> 10k
- R5: value 100 -> 10k
- R6: value 1k -> 10k
Connections:
- net VBUS_MON is gone; now on an unnamed net: R6.2
- net D+: now also U3.6 (NC); no longer J1.A6 (D+), J1.B6 (D+)
- net D-: now also U3.7 (NC); no longer J1.A7 (D-), J1.B7 (D-)
- net Earth: now also C18.2, R3.1, D37.1 (A1), TH1.2, U2.18 (AGND), U2.5 (PGND), U3.3 (G), U3.8 (G)
- net SCL: now also U2.16 (SCL)
- net SDA: now also U2.15 (SDA)
- net VBUS: now also C13.1, D37.2 (A2), U2.2 (IN); no longer C15.1, C17.1, R6.1
- net VSYS: no longer C18.1
- net at C12.1: now also U2.3 (PMID)
- net at J1.A5 (CC1): now also U3.1 (IO1)
- net at C14.1: now also R5.2, U2.19 (VCC); no longer R4.1
- net at J1.B5 (CC2): now also U3.2 (IO2)
- net at C15.2: now also U2.6 (BST); no longer R5.2
- net at C16.1: now also C17.1, L3.2, U2.13 (SYS)
- net BATT: no longer names the net of BT1.1 (+)
- net BATT: now also F1.1; no longer BT2.1 (+)
- net VBUS_EN: no longer names the net of R3.2
- net VBUS_EN: now also U2.17 (~{RST})
- new net: C18.1, F1.2, F2.2, U2.12 (BATTSNS), U2.14 (BATT)
- new net: R6.1, U2.11 (STAT)
- new net: R5.1, U2.9 (PG)
- new net: C15.1, L3.1, U2.4 (SW)
- new net: R4.1, TH1.1, U2.10 (NTC)
- new net: R4.2, U2.7 (VRNTC)
- new net: J1.A6 (D+), J1.B6 (D+), U3.5 (IO4)
- new net: J1.A7 (D-), J1.B7 (D-), U3.4 (IO3)
- new net: BT2.1 (+), F2.1
- new net CC1: U2.1 (CC1), U3.10 (NC)
- new net CC2: U2.22 (CC2), U3.9 (NC)
- no-connect marks 18 -> 6
Other:
- note added: "Fuses used: PTS18126V260"
- note removed: "3V5 - 4V5"
- note removed: "D+ and D- pins are not used All the settings are handled from MCU through I2C It's recommended to disable D+/D- detection together with Maxcharge and HVDCP in the REG02 register"
- note removed: "Recommended value for R_{1} at 12V output is 240k R_{2} value can be calculated as R_{2} = R_{1} / ((V_{OUT} / 1.24) - 1)"
- moved on the sheet: C29, C30, TP5, U6

Commit message: Schematic update
Removed one battery, changed battery fuse to correct one. Fixed OLED connector
Parts:
- removed BT1: BATT_1, symbol Device:Battery_Cell
- removed F1: F_BATT_1, symbol Device:Fuse_Small
- BT2: value BATT_2 -> BATT
- F2: value F_BATT_2 -> 2016L500DR
Other:
- note removed: "Fuses used: PTS18126V260"
- moved on the sheet: BT2, C18, F2

Commit message: PCB Layout mostly completed
Still have to finish LEDs layout on back side
Parts:
- BT2: footprint (none) -> Connector_JST:JST_SH_BM02B-SRSS-TB_1x02-1MP_P1.00mm_Vertical
- C12, C16, C17, C18: footprint (none) -> Capacitor_SMD:C_0805_2012Metric
- C13, C14, C15, C29, C30: footprint (none) -> Capacitor_SMD:C_0603_1608Metric
- D37: footprint (none) -> Diode_SMD:D_SOD-123F
- F2: footprint (none) -> Fuse:Fuse_2010_5025Metric
- J1: footprint (none) -> Connector_USB:USB_C_Receptacle_Molex_105450-0101
- L3: footprint (none) -> Inductor_SMD:L_1210_3225Metric
- R3, R5, R6, TH1: footprint (none) -> Resistor_SMD:R_0402_1005Metric
- R4: footprint (none) -> Resistor_SMD:R_0603_1608Metric
- TP1, TP5: footprint (none) -> TestPoint:TestPoint_Pad_D2.0mm
Connections:
- net CC1: now also U3.9 (NC); no longer U3.10 (NC)
- net CC2: now also U3.10 (NC); no longer U3.9 (NC)
- net VSYS: now also C16.1, C17.1, L3.2, U2.13 (SYS)
- net at J1.A5 (CC1): now also U3.2 (IO2); no longer U3.1 (IO1)
- net USB_D+: now reaches J1.A6 (D+), J1.B6 (D+)
- net USB_D+: now also U3.4 (IO3); no longer U3.5 (IO4)
- net USB_D-: now reaches J1.A7 (D-), J1.B7 (D-)
- net USB_D-: now also U3.5 (IO4); no longer U3.4 (IO3)
- net at J1.B5 (CC2): now also U3.1 (IO1); no longer U3.2 (IO2)
Other:
- moved on the sheet: U3

Commit message: PCB Optimalizations
Parts:
- added TP2: TP_VSYS, TestPoint:TestPoint_Pad_D2.0mm, symbol Connector:TestPoint_Small
Connections:
- net VSYS: now also TP2.1
Changed lines of the file:
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@@
   (junction (at 105.41 31.75) (diameter 0) (color 0 0 0 0)
+  )
+  (junction (at 109.22 116.84) (diameter 0) (color 0 0 0 0)
   )
   (junction (at 135.89 31.75) (diameter 0) (color 0 0 0 0)
@@
     (stroke (width 0) (type default))
   )
+  (wire (pts (xy 109.22 116.84) (xy 109.22 121.92))
+    (stroke (width 0) (type default))
+  )
   (wire (pts (xy 106.68 130.81) (xy 106.68 129.54))
     (stroke (width 0) (type default))
@@
     (stroke (width 0) (type default))
   )
-  (wire (pts (xy 109.22 121.92) (xy 109.22 119.38))
-    (stroke (width 0) (type default))
-  )
   (wire (pts (xy 35.56 82.55) (xy 35.56 83.82))
     (stroke (width 0) (type default))
@@
     (stroke (width 0) (type default))
   )
+  (wire (pts (xy 109.22 111.76) (xy 109.22 116.84))
+    (stroke (width 0) (type default))
+  )
   (wire (pts (xy 40.64 124.46) (xy 43.18 124.46))
     (stroke (width 0) (type default))
@@
     (stroke (width 0) (type default))
   )
-  (wire (pts (xy 147.32 27.94) (xy 147.32 24.13))
-    (stroke (width 0) (type default))
-  )
   (wire (pts (xy 40.64 138.43) (xy 43.18 138.43))
     (stroke (width 0) (type default))
@@
   )
   (wire (pts (xy 113.03 31.75) (xy 105.41 31.75))
+    (stroke (width 0) (type default))
+  )
+  (wire (pts (xy 147.32 24.13) (xy 147.32 27.94))
     (stroke (width 0) (type default))
   )
@@
     )
   )
+  (symbol (lib_id "Connector:TestPoint_Small") (at 109.22 116.84 180) (unit 1)
+    (in_bom yes) (on_board yes) (dnp no) (fields_autoplaced)
+    (property "Reference" "TP2" (at 110.49 115.57 0)
+      (effects (font (size 1.27 1.27)) (justify right))
+    )
+    (property "Value" "TP_VSYS" (at 110.49 118.11 0)
+      (effects (font (size 1.27 1.27)) (justify right))
+    )
+    (property "Footprint" "TestPoint:TestPoint_Pad_D2.0mm" (at 104.14 116.84 0)
+      (effects (font (size 1.27 1.27)) hide)
+    )
+    (property "Datasheet" "~" (at 104.14 116.84 0)
+      (effects (font (size 1.27 1.27)) hide)
+    )
+    (pin "1")
+    (instances
+      (project "Aitken"
+        (path "/b70621e2-23d0-406f-b359-5b7c90496935/b637dce6-9faa-48d7-ac20-34c7af1e210c"
+          (reference "TP2") (unit 1)
+        )
+      )
+    )
+  )
   (symbol (lib_id "Device:C_Small") (at 96.52 125.73 0) (unit 1)
     (in_bom yes) (on_board yes) (dnp no) (fields_autoplaced)
@@
     )
   )
-  (symbol (lib_id "more_power:VSYS") (at 109.22 119.38 0) (unit 1)
-    (in_bom yes) (on_board yes) (dnp no) (fields_autoplaced)
-    (property "Reference" "#PWR062" (at 109.22 123.19 0)
-      (effects (font (size 1.27 1.27)) hide)
-    )
-    (property "Value" "VSYS" (at 109.22 115.57 0)
-      (effects (font (size 1.27 1.27)))
-    )
-    (property "Footprint" "" (at 109.22 119.38 0)
-      (effects (font (size 1.27 1.27)) hide)
-    )
-    (property "Datasheet" "" (at 109.22 119.38 0)
-      (effects (font (size 1.27 1.27)) hide)
-    )
+  (symbol (lib_id "more_power:VSYS") (at 109.22 111.76 0) (unit 1)
+    (in_bom yes) (on_board yes) (dnp no) (fields_autoplaced)
+    (property "Reference" "#PWR062" (at 109.22 115.57 0)
+      (effects (font (size 1.27 1.27)) hide)
+    )
+    (property "Value" "VSYS" (at 109.22 107.95 0)
+      (effects (font (size 1.27 1.27)))
+    )
+    (property "Footprint" "" (at 109.22 111.76 0)
+      (effects (font (size 1.27 1.27)) hide)
+    )
+    (property "Datasheet" "" (at 109.22 111.76 0)
+      (effects (font (size 1.27 1.27)) hide)
+    )

Commit message: Auto stash before merge of "latest" and "origin/latest"
Parts:
- added TP2: TP_VSYS, TestPoint:TestPoint_Pad_D2.0mm, symbol Connector:TestPoint_Small
- J1: footprint Connector_USB:USB_C_Receptacle_Molex_105450-0101 -> USB4085:GCT_USB4085-GF-A_REVB
Connections:
- net VSYS: now also TP2.1
Changed lines of the file:
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@@
   (junction (at 74.93 140.97) (diameter 0) (color 0 0 0 0)
+  )
+  (junction (at 109.22 116.84) (diameter 0) (color 0 0 0 0)
   )
   (junction (at 34.29 163.83) (diameter 0) (color 0 0 0 0)
@@
     (stroke (width 0) (type default))
   )
+  (wire (pts (xy 109.22 116.84) (xy 109.22 114.3))
+    (stroke (width 0) (type default))
+  )
   (wire (pts (xy 58.42 67.31) (xy 74.93 67.31))
     (stroke (width 0) (type default))
@@
   )
   (wire (pts (xy 72.39 132.08) (xy 73.66 132.08))
+    (stroke (width 0) (type default))
+  )
+  (wire (pts (xy 109.22 121.92) (xy 109.22 116.84))
     (stroke (width 0) (type default))
   )
@@
       (effects (font (size 1.27 1.27)))
     )
-    (property "Footprint" "Connector_USB:USB_C_Receptacle_Molex_105450-0101" (at 39.37 59.69 0)
+    (property "Footprint" "USB4085:GCT_USB4085-GF-A_REVB" (at 39.37 59.69 0)
       (effects (font (size 1.27 1.27)) hide)
     )
@@
     )
   )
+  (symbol (lib_id "Connector:TestPoint_Small") (at 109.22 116.84 180) (unit 1)
+    (in_bom yes) (on_board yes) (dnp no) (fields_autoplaced)
+    (property "Reference" "TP2" (at 110.49 116.205 0)
+      (effects (font (size 1.27 1.27)) (justify right))
+    )
+    (property "Value" "TP_VSYS" (at 110.49 118.745 0)
+      (effects (font (size 1.27 1.27)) (justify right))
+    )
+    (property "Footprint" "TestPoint:TestPoint_Pad_D2.0mm" (at 104.14 116.84 0)
+      (effects (font (size 1.27 1.27)) hide)
+    )
+    (property "Datasheet" "~" (at 104.14 116.84 0)
+      (effects (font (size 1.27 1.27)) hide)
+    )
+    (pin "1")
+    (instances
+      (project "Aitken"
+        (path "/b70621e2-23d0-406f-b359-5b7c90496935/b637dce6-9faa-48d7-ac20-34c7af1e210c"
+          (reference "TP2") (unit 1)
+        )
+      )
+    )
+  )
   (symbol (lib_id "power:VBUS") (at 63.5 30.48 0) (unit 1)
     (in_bom yes) (on_board yes) (dnp no) (fields_autoplaced)
@@
     )
   )
-  (symbol (lib_id "more_power:VSYS") (at 109.22 111.76 0) (unit 1)
-    (in_bom yes) (on_board yes) (dnp no) (fields_autoplaced)
-    (property "Reference" "#PWR062" (at 109.22 115.57 0)
-      (effects (font (size 1.27 1.27)) hide)
-    )
-    (property "Value" "VSYS" (at 109.22 107.95 0)
+  (symbol (lib_id "more_power:VSYS") (at 109.22 114.3 0) (unit 1)
+    (in_bom yes) (on_board yes) (dnp no) (fields_autoplaced)
+    (property "Reference" "#PWR062" (at 109.22 118.11 0)
+      (effects (font (size 1.27 1.27)) hide)
+    )
+    (property "Value" "VSYS" (at 109.22 110.49 0)
       (effects (font (size 1.27 1.27)))
     )
-    (property "Footprint" "" (at 109.22 111.76 0)
-      (effects (font (size 1.27 1.27)) hide)
-    )
-    (property "Datasheet" "" (at 109.22 111.76 0)
-      (effects (font (size 1.27 1.27)) hide)
-    )
+    (property "Footprint" "" (at 109.22 114.3 0)
+      (effects (font (size 1.27 1.27)) hide)
+    )
+    (property "Datasheet" "" (at 109.22 114.3 0)
+      (effects (font (size 1.27 1.27)) hide)
+    )
