File: Electronics/Aitken.kicad_pcb (KiCad board)
At the start: 4 copper layers, 55 x 65 mm, 118 parts, among them J1 USB_C_Receptacle_USB2.0, J2 OLED_CONN, J3 UART_CONN, SW2 PEC12, SW4 MCU_EN, U1 ESP32-C4FH4, U2 MP2722, U3 TPD4E02B04DQA, U4 LIS3MDL, U5 LSM6DS3, U6 NCP186AMX330TAG, U7 KTD2801, U8 KTD2801, U9 KTD2801, Y1 40MHz

Commit message: Basic PCB layout finished
Parts:
- moved D16 83.4 mm to (200.1, 79.3), turned to 90 degrees
- moved D15 82.8 mm to (185.3, 79.4), turned to -90 degrees
- moved D4 72.8 mm to (167.2, 86.5)
- moved D3 70.1 mm to (170.1, 101.4)
- moved D2 69.5 mm to (170.1, 114.3)
- moved D5 68.1 mm to (174.7, 79.2), turned to 90 degrees
- moved D1 65.8 mm to (167.2, 129.9)
- moved D17 64.5 mm to (197.4, 93.7), turned to 90 degrees
- moved D14 63.6 mm to (188.2, 93.9), turned to -90 degrees
- moved D9 60.2 mm to (174.7, 123.8)
- moved D10 58.4 mm to (174.7, 137.4)
- moved D8 57.5 mm to (180.9, 113.9)
- moved D7 56.9 mm to (180.9, 102.2)
- moved D6 54.6 mm to (174.7, 92.6)
- moved D25 52.9 mm to (209.8, 79.2), turned to 90 degrees
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Routing:
- net Net-(D21-A): track 2.18 -> 29.6 mm, vias 0 -> 1
- net unconnected-(J1-SHIELD-PadS1): track 0.00 -> 19.4 mm
- net Net-(D1-A): track 2.26 -> 20.9 mm, vias 1 -> 2
- net Net-(D15-K): track 0.00 -> 15.8 mm
- net Net-(D1-K): track 0.00 -> 14.6 mm
- net Net-(D3-K): track 0.00 -> 13.9 mm
- net Net-(D12-K): track 0.00 -> 13.8 mm
- net Net-(D23-K): track 0.00 -> 13.8 mm
- net Net-(D13-K): track 0.00 -> 13.6 mm
- net Net-(D14-K): track 0.00 -> 13.6 mm
- net Net-(D11-K): track 0.00 -> 13.6 mm
- net Net-(D19-K): track 0.00 -> 13.5 mm
- net Net-(D17-K): track 0.00 -> 13.5 mm
- net Net-(D16-K): track 0.00 -> 13.3 mm
- net Net-(D24-K): track 0.00 -> 12.9 mm
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- added copper zone on F.Cu, net +3V3
- added copper zone on B.Cu, net Earth
- added copper zone on F.Cu, net Net-(BT2-+)
- added copper zone on F.Cu, net Net-(U7-LX)
- added copper zone on F.Cu, net Net-(U8-LX)
- added copper zone on F.Cu, net Net-(U9-LX)
- added copper zone on F.Cu, net VSYS
Other:
- board text added: "3V3"
- board text added: "GND"
- board text added: "RX"
- board text added: "SCL"
- board text added: "SDA"
- board text added: "TX"

Commit message: PCB Optimalizations
Routing:
- net VSYS: track 100.6 -> 94.9 mm, vias 0 -> 9
- net /MCU/ENC_S: track 29.4 -> 34.1 mm
- net Earth: track 62.4 -> 65.4 mm, vias 69 -> 74
- net Net-(U2-STAT): track 5.12 -> 8.09 mm
- net Net-(D17-K): track 13.5 -> 16.3 mm
- net Net-(U2-BATT): track 10.8 -> 8.86 mm
- net Net-(U2-NTC): track 17.1 -> 15.4 mm
- net Net-(U2-SW): track 9.25 -> 9.91 mm
- added copper zone on F.Cu, net Net-(U2-BATT)
- added copper zone on B.Cu, net VSYS

Commit message: Changed USB port
Parts:
- added TP2: TP_VSYS, TestPoint:TestPoint_Pad_D2.0mm, F.Cu at (200.4, 115.5)
- J1: footprint Connector_USB:USB_C_Receptacle_Molex_105450-0101 -> USB4085:GCT_USB4085-GF-A_REVB
- moved J1 2.56 mm to (192.6, 77.5)
Routing:
- net unconnected-(J1-SHIELD-PadS1): track 19.4 -> 0.00 mm
- net /Power management/USB_D+: track 5.03 -> 13.6 mm, vias 2 -> 0
- net /Power management/USB_D-: track 5.28 -> 13.6 mm, vias 2 -> 0
- net VBUS: track 29.6 -> 33.4 mm, vias 4 -> 3
- net Net-(J1-CC2): track 6.78 -> 9.79 mm, vias 2 -> 1
- net Net-(J1-CC1): track 3.77 -> 4.98 mm, vias 0 -> 1
- net Earth: track 65.4 -> 65.1 mm, vias 74 -> 72

Commit message: Cosmetic PCB changes
Added silkscreen labels and logo. Other minor fixes
Parts:
- moved TP2 22.4 mm to (179.7, 124.0)
- moved H3 0.36 mm to (215.6, 136.6)
- moved AE1 0.23 mm to (180.0, 78.8)
- moved C9 0.23 mm to (179.0, 81.0)
- moved L2 0.23 mm to (178.6, 82.8)
- moved H4 0.20 mm to (169.0, 136.6)
Routing:
- net Earth: track 65.1 -> 75.2 mm, vias 72 -> 82
- net +3V3: track 46.7 -> 39.9 mm, vias 16 -> 17
- net /Power management/USB_D-: track 13.6 -> 6.97 mm
- net /Power management/USB_D+: track 13.6 -> 7.01 mm
- net TX: track 37.4 -> 34.7 mm
- net Net-(D6-K): track 10.1 -> 12.2 mm
- net Net-(J1-CC2): track 9.79 -> 11.1 mm
- net CC1: track 7.59 -> 7.05 mm
- net /MCU/ENC_B: vias 2 -> 1
- net /MCU/ENC_A: vias 2 -> 1
- added copper zone on F.Cu, net Net-(U2-PMID)
- added copper zone on F.Cu, net Net-(U2-SW)
- added copper zone on F.Cu, net VBUS
Other:
- board text added: "Antenna"
- board text added: "Battery"
- board text added: "OLED"
- board text added: "V_{BUS}"
- board text added: "V_{SYS}"
- board text added: "Version 1.0 2023-11-30"

Commit message: Fixed antenna
Parts:
- moved C5 5.07 mm to (173.1, 83.3)
- moved C6 2.05 mm to (175.4, 82.6), turned to -90 degrees
- moved L2 1.18 mm to (178.4, 83.9)
- moved C8 1.15 mm to (178.9, 85.6)
- moved C9 1.15 mm to (178.9, 82.1)
- moved C7 0.42 mm to (176.7, 84.4)
- moved AE1 0.18 mm to (179.9, 78.9)
Connections:
- AE1 pad 2: Earth -> unconnected-(AE1-Shield-Pad2)
Routing:
- net Earth: track 75.2 -> 72.7 mm, vias 82 -> 106
- net /MCU/LNA_IN: track 3.86 -> 2.49 mm
- net Net-(AE1-A): track 3.56 -> 4.53 mm
- net Net-(D12-K): track 13.8 -> 13.9 mm, vias 0 -> 1
Other:
- board text added: "RESET"

Commit message: Fixed crystal
Parts:
- Y1: footprint Crystal:Crystal_SMD_2520-4Pin_2.5x2.0mm -> Crystal:Crystal_SMD_3225-4Pin_3.2x2.5mm
- moved C10 4.75 mm to (189.1, 84.4)
- moved Y1 0.79 mm to (185.1, 86.0), turned to 90 degrees
Connections:
- Y1 pad 2: /MCU/XTAL_IN -> Earth
- Y1 pad 3: Earth -> /MCU/XTAL_IN
- Y1 pad 4: (no net) -> Earth
Routing:
- net /MCU/XTAL_IN: track 3.37 -> 6.51 mm
- net Earth: track 72.7 -> 74.4 mm, vias 106 -> 105
- net /MCU/XTAL_N: track 13.9 -> 12.3 mm
