File: Electronics/Aitken.kicad_pcb (KiCad board)
At the start: 4 copper layers, 55 x 65 mm, 119 parts, among them J1 USB_C_Receptacle_USB2.0, J2 OLED_CONN, J3 UART_CONN, SW2 PEC12, SW4 MCU_EN, U1 ESP32-C4FH4, U2 MP2722, U3 TPD4E02B04DQA, U4 LIS3MDL, U5 LSM6DS3, U6 NCP186AMX330TAG, U7 KTD2801, U8 KTD2801, U9 KTD2801, Y1 40MHz

Commit message: Minor fixes
Parts:
- moved C12 1.03 mm to (194.3, 94.8)
- moved R4 0.54 mm to (191.6, 95.6)
- moved TH1 0.54 mm to (191.1, 94.1)
- moved JP2 0.43 mm to (188.0, 95.6)
Routing:
- net Net-(U2-NTC): track 15.4 -> 14.4 mm
- net Net-(U2-PMID): track 3.52 -> 4.55 mm
- net Earth: track 74.4 -> 73.5 mm, vias 105 -> 112
- net /Sensors/MAG_ADD: track 6.35 -> 5.75 mm
- net Net-(U2-VRNTC): track 12.6 -> 13.1 mm
