File: Electronics/mcu.kicad_sch (KiCad schematic)
At the start: 34 parts, among them J2 OLED_CONN, J3 UART_CONN, SW2 PEC12, SW4 MCU_EN, Y1 40MHz, Y2 32kHz

Commit message: Schematic update
Added correct values for crystal capacitors, added net labels and minor cleanup
Parts:
- added R36, R37: 470R, symbol Device:R_Small
- C10, C11: value 10p -> 11p
- C34, C35: value ? -> 10p
Connections:
- net RX: now also R36.1; no longer U1.27 (U0RXD)
- net TX: now also R37.1; no longer U1.28 (U0TXD)
- net ENC_A: now reaches R31.2, SW2.A, U1.15 (GPIO9)
- net ENC_B: now reaches R32.2, SW2.B, U1.16 (GPIO10)
- net ENC_S: now reaches R30.1, SW2.S1, U1.8 (GPIO3)
- net XTAL_32K_IN: now reaches C34.1, R35.1, Y2.2
- net XTAL_32K_P: now reaches R35.2, U1.4 (XTAL_32K_P)
- net XTAL_IN: now reaches C11.1, R1.1, Y1.2
- net XTAL_P: now reaches R1.2, U1.30 (XTAL_P)
- net XTAL_32K_N: now reaches C35.1, U1.5 (XTAL_32K_N), Y2.1
- net ~{CHIP_EN}: now reaches C36.2, R2.1, SW4.2, U1.7 (~{CHIP_EN})
- net LNA_IN: now reaches C8.1, L2.2, U1.1 (LNA_IN)
- net XTAL_N: now reaches C10.1, U1.29 (XTAL_N), Y1.1
- new net ESP32_RX: R36.2, U1.27 (U0RXD)
- new net ESP_32TX: R37.2, U1.28 (U0TXD)
Other:
- note added: "MC-405 32"
- note added: "RH100-40.000-16"
- moved on the sheet: C10, C11, C34, C35, R1, R2, R28, R29, R35, Y1, Y2

Commit message: Power and lights update
Changed STUSB4500 + BQ25895 to MP2722. Changed Lights power supply, now it's split up to 3 LED drivers - KTD2801 as 10s1p. Added fuses to each battery. Added ESD protection. Fixed CHIP_EN pin name on ESP32-C3 and pull-up resistor on I2C lines.
Parts:
- U1: value ~ -> ESP32-C4FH4
Connections:
- net SCL: no longer R29.2
- net SDA: now also R29.2
- net ESP_32TX renamed ESP32_TX
- net ~{CHIP_EN} renamed CHIP_EN

Commit message: Schematic update
Removed one battery, changed battery fuse to correct one. Fixed OLED connector
Parts:
- AE1: value BL_WIFI_ANT -> ANT3216A063R2400A
Connections:
- net +3V3: now also J2.1 (Pin_1); no longer J2.4 (Pin_4)
- net Earth: now also J2.2 (Pin_2); no longer J2.1 (Pin_1)
- net SCL: now also J2.3 (Pin_3); no longer J2.2 (Pin_2)
- net SDA: now also J2.4 (Pin_4); no longer J2.3 (Pin_3)
Other:
- moved on the sheet: C36, R2, SW4

Commit message: PCB Layout mostly completed
Still have to finish LEDs layout on back side
Parts:
- removed C34, C35: 10p, symbol Device:C_Small
- removed R35: 22R, symbol Device:R_Small
- removed Y2: 32kHz, symbol Device:Crystal_GND3_Small
- AE1: value ANT3216A063R2400A -> 2450AT18x0100; footprint (none) -> RF_Antenna:Johanson_2450AT18x100
- C1, C10, C11, C2, C3, C36, C6, C7, C8, C9: footprint (none) -> Capacitor_SMD:C_0402_1005Metric
- C4, C5: footprint (none) -> Capacitor_SMD:C_0603_1608Metric
- J2, J3: footprint (none) -> Connector_PinHeader_2.54mm:PinHeader_1x04_P2.54mm_Vertical
- L1, L2: footprint (none) -> Inductor_SMD:L_0402_1005Metric
- R1, R2, R28, R29, R30, R31, R32, R34, R36, R37: footprint (none) -> Resistor_SMD:R_0402_1005Metric
- R33: value 1k -> 5k1; footprint (none) -> Resistor_SMD:R_0402_1005Metric
- SW2: footprint (none) -> Rotary_Encoder:RotaryEncoder_Bourns_Vertical_PEC12R-3xxxF-Sxxxx
- SW4: footprint (none) -> Button_Switch_SMD:SW_Push_1P1T_NO_6x6mm_H9.5mm
- Y1: footprint (none) -> Crystal:Crystal_SMD_2520-4Pin_2.5x2.0mm
Connections:
- net XTAL_32K_N: no longer names the net of U1.5 (XTAL_32K_N)
- net XTAL_32K_P: no longer names the net of U1.4 (XTAL_32K_P)
- no-connect marks 4 -> 6
Other:
- note removed: "MC-405 32"

Commit message: Fixed antenna
Connections:
- net Earth: no longer AE1.2 (Shield)
- no-connect marks 6 -> 7
Other:
- moved on the sheet: AE1
Changed lines of the file:
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@@
   (junction (at 140.97 53.34) (diameter 0) (color 0 0 0 0)
   )
-  (junction (at 74.93 80.01) (diameter 0) (color 0 0 0 0)
-  )
   (junction (at 158.75 83.82) (diameter 0) (color 0 0 0 0)
   )
@@
   (junction (at 154.94 119.38) (diameter 0) (color 0 0 0 0)
   )
+  (no_connect (at 66.04 74.93))
   (no_connect (at 105.41 130.81))
   (no_connect (at 105.41 133.35))
@@
     (stroke (width 0) (type default))
   )
-  (wire (pts (xy 69.85 77.47) (xy 69.85 80.01))
-    (stroke (width 0) (type default))
-  )
   (wire (pts (xy 92.71 53.34) (xy 102.87 53.34))
     (stroke (width 0) (type default))
@@
     (stroke (width 0) (type default))
   )
-  (wire (pts (xy 69.85 72.39) (xy 69.85 74.93))
-    (stroke (width 0) (type default))
-  )
   (wire (pts (xy 87.63 102.87) (xy 87.63 96.52))
     (stroke (width 0) (type default))
@@
     (stroke (width 0) (type default))
   )
-  (wire (pts (xy 69.85 80.01) (xy 74.93 80.01))
-    (stroke (width 0) (type default))
-  )
   (wire (pts (xy 148.59 81.28) (xy 165.1 81.28))
     (stroke (width 0) (type default))
@@
     (stroke (width 0) (type default))
   )
-  (wire (pts (xy 69.85 72.39) (xy 74.93 72.39))
+  (wire (pts (xy 66.04 72.39) (xy 74.93 72.39))
     (stroke (width 0) (type default))
   )
@@
     )
   )
-  (symbol (lib_id "Device:Antenna_Shield") (at 64.77 74.93 90) (mirror x) (unit 1)
+  (symbol (lib_id "Device:Antenna_Shield") (at 60.96 72.39 90) (mirror x) (unit 1)
     (in_bom yes) (on_board yes) (dnp no)
-    (property "Reference" "AE1" (at 62.23 71.12 90)
+    (property "Reference" "AE1" (at 58.42 68.58 90)
       (effects (font (size 1.27 1.27)))
     )
-    (property "Value" "2450AT18x0100" (at 62.23 78.74 90)
+    (property "Value" "2450AT18x0100" (at 58.42 76.2 90)
       (effects (font (size 0.75 0.75)))
     )
-    (property "Footprint" "RF_Antenna:Johanson_2450AT18x100" (at 62.23 74.93 0)
-      (effects (font (size 1.27 1.27)) hide)
-    )
-    (property "Datasheet" "~" (at 62.23 74.93 0)
-      (effects (font (size 1.27 1.27)) hide)
-    )
+    (property "Footprint" "RF_Antenna:Johanson_2450AT18x100" (at 58.42 72.39 0)
+      (effects (font (size 1.27 1.27)) hide)
+    )
+    (property "Datasheet" "~" (at 58.42 72.39 0)
+      (effects (font (size 1.27 1.27)) hide)
+    )

Commit message: Fixed crystal
Parts:
- removed Y1: 40MHz, Crystal:Crystal_SMD_2520-4Pin_2.5x2.0mm, symbol Device:Crystal_GND3_Small
- added Y1: 40MHz, Crystal:Crystal_SMD_3225-4Pin_3.2x2.5mm, symbol Device:Crystal_GND24_Small
Connections:
- net Earth: now also Y1.2, Y1.4
- net XTAL_IN: now also Y1.3
- net XTAL_N: now also Y1.1
Other:
- note removed: "RH100-40.000-16"
- moved on the sheet: C10, C11
